File: PCB/controller/controller.kicad_pcb (KiCad board)
At the start: 2 copper layers, 18 parts, among them X1 Switch, Y1 Switch

Commit message: doin stuffs
Parts:
- removed A1: RaspberryPi_Pico_W, Module:RaspberryPi_Pico_W_SMD_HandSolder
- removed Bk1, Bk2, Home1, L1, Options1, R1, ZL1, ZR1: Switch, Button_Switch_SMD:SW_Push_1P1T_NO_CK_KSC6xxJ
- added D1: 1N4148, Diode_THT:D_DO-35_SOD27_P7.62mm_Horizontal, F.Cu at (129.7, 90.8)
- added D10: 1N4148, Diode_THT:D_DO-35_SOD27_P7.62mm_Horizontal, F.Cu at (206.5, 111.8)
- added D11: 1N4148, Diode_THT:D_DO-35_SOD27_P7.62mm_Horizontal, F.Cu at (224.5, 88.0)
- added D12: 1N4148, Diode_THT:D_DO-35_SOD27_P7.62mm_Horizontal, F.Cu at (206.0, 84.5)
- added D2: 1N4148, Diode_THT:D_DO-35_SOD27_P7.62mm_Horizontal, F.Cu at (157.0, 91.3)
- added D3: 1N4148, Diode_THT:D_DO-35_SOD27_P7.62mm_Horizontal, F.Cu at (149.3, 111.3)
- added D4: 1N4148, Diode_THT:D_DO-35_SOD27_P7.62mm_Horizontal, F.Cu at (130.2, 103.8)
- added D9: 1N4148, Diode_THT:D_DO-35_SOD27_P7.62mm_Horizontal, F.Cu at (225.5, 103.5)
- added R2: THB001P, ScottoKeebs_Miscellaneous:THB001P_CNK, F.Cu at (225.1, 115.9)
- added U1: Raspberry_Pi_Pico, ScottoKeebs_MCU:Raspberry_Pi_Pico, F.Cu at (179.2, 108.5)
- moved Y1 145.6 mm to (204.0, 98.0), turned to 90 degrees
- moved X1 144.3 mm to (212.0, 91.6), turned to 90 degrees
- moved A2 142.1 mm to (220.0, 97.5), turned to -90 degrees
- moved BT1 82.3 mm to (163.4, 145.5), turned to 0 degrees
- moved D_Down1 50.5 mm to (143.3, 106.4), turned to 90 degrees
- moved D_Left1 48.5 mm to (136.3, 97.7), turned to 90 degrees
- moved B1 46.8 mm to (212.0, 105.9), turned to -90 degrees
- moved D_UP1 38.8 mm to (143.3, 89.2), turned to -90 degrees
- moved D_right1 31.8 mm to (150.3, 97.3), turned to -90 degrees
Connections:
- A2 pad 1: Net-(A1-3V3) -> Net-(U1-GPIO6)
- B1 pad 1: Net-(A1-3V3) -> Net-(U1-GPIO7)
- D_Down1 pad 1: Net-(A1-3V3) -> Net-(U1-GPIO8)
- D_Left1 pad 1: Net-(A1-3V3) -> Net-(U1-GPIO9)
- D_UP1 pad 1: Net-(A1-3V3) -> Net-(U1-GPIO6)
- D_right1 pad 1: Net-(A1-3V3) -> Net-(U1-GPIO7)
- X1 pad 1: Net-(A1-3V3) -> Net-(U1-GPIO8)
- Y1 pad 1: Net-(A1-3V3) -> Net-(U1-GPIO9)
Routing:
- net Net-(BT1-+): track 17.4 -> 124.3 mm
- net Net-(D1-K): track 0.00 -> 58.5 mm
- net Net-(D10-K): track 0.00 -> 58.3 mm
- net Net-(BT1--): track 11.5 -> 38.6 mm
- net Net-(D1-A): track 0.00 -> 4.54 mm
- net Net-(D3-A): track 0.00 -> 3.62 mm
- net Net-(D2-A): track 0.00 -> 3.51 mm
- net Net-(D4-A): track 0.00 -> 3.41 mm

Commit message: more work
Parts:
- removed BT1: Battery_Cell, Battery:BatteryHolder_Bulgin_BX0034_1xAAA
- removed R2: THB001P, ScottoKeebs_Miscellaneous:THB001P_CNK
- removed U1: Raspberry_Pi_Pico, ScottoKeebs_MCU:Raspberry_Pi_Pico
- added A1: Adafruit_Feather_32u4_BluefruitLE, Module:Adafruit_Feather, F.Cu at (86.9, 66.5)
- added stick1: THB001P, ScottoKeebs_Miscellaneous:THB001P_CNK, F.Cu at (59.6, 69.9)
- added stick2: THB001P, ScottoKeebs_Miscellaneous:THB001P_CNK, F.Cu at (126.5, 108.5)
- moved D9 115.7 mm to (111.0, 87.0), turned to 0 degrees
- moved D11 113.8 mm to (111.0, 80.0), turned to 0 degrees
- moved D12 92.2 mm to (114.0, 90.0), turned to 0 degrees
- moved D10 85.4 mm to (123.0, 94.0), turned to 0 degrees
- moved D2 82.8 mm to (75.0, 103.0), turned to 0 degrees
- moved Y1 80.1 mm to (125.6, 81.5), turned to 0 degrees
- moved B1 79.4 mm to (134.5, 88.5), turned to 0 degrees
- moved X1 79.4 mm to (134.5, 74.5), turned to 0 degrees
- moved A2 78.3 mm to (143.4, 81.5), turned to 0 degrees
- moved D_Left1 78.2 mm to (60.1, 115.0), turned to 0 degrees
- moved D_UP1 76.7 mm to (69.0, 108.0), turned to 0 degrees
- moved D_Down1 75.9 mm to (69.1, 122.0), turned to 0 degrees
- moved D_right1 74.6 mm to (77.9, 115.0), turned to 0 degrees
- moved D4 71.2 mm to (59.0, 103.0)
- moved D1 63.4 mm to (67.0, 100.0)
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Connections:
- A2 pad 1: Net-(U1-GPIO6) -> col2
- B1 pad 1: Net-(U1-GPIO7) -> col2
- D1 pad 1: Net-(D1-K) -> row0
- D10 pad 1: Net-(D10-K) -> row1
- D11 pad 1: Net-(D10-K) -> row2
- D12 pad 1: Net-(D10-K) -> row3
- D2 pad 1: Net-(D1-K) -> row1
- D3 pad 1: Net-(D1-K) -> row2
- D4 pad 1: Net-(D1-K) -> row3
- D9 pad 1: Net-(D10-K) -> row0
- D_Down1 pad 1: Net-(U1-GPIO8) -> col0
- D_Left1 pad 1: Net-(U1-GPIO9) -> col0
- D_UP1 pad 1: Net-(U1-GPIO6) -> col0
- D_right1 pad 1: Net-(U1-GPIO7) -> col0
- X1 pad 1: Net-(U1-GPIO8) -> col2
- Y1 pad 1: Net-(U1-GPIO9) -> col2
Routing:
- net 3.3v: track 0.00 -> 192.3 mm, vias 0 -> 1
- net col0: track 0.00 -> 161.3 mm
- net row3: track 0.00 -> 155.7 mm
- net gnd: track 0.00 -> 125.1 mm
- net Net-(BT1-+): track 124.3 -> 0.00 mm
- net row2: track 0.00 -> 118.3 mm, vias 0 -> 1
- net row1: track 0.00 -> 103.5 mm, vias 0 -> 1
- net y1: track 0.00 -> 68.3 mm
- net Net-(D1-K): track 58.5 -> 0.00 mm
- net Net-(D10-K): track 58.3 -> 0.00 mm
- net y2: track 0.00 -> 56.9 mm
- net col2: track 0.00 -> 56.6 mm
- net x1: track 0.00 -> 47.5 mm
- net row0: track 0.00 -> 43.3 mm
- net x2: track 0.00 -> 38.9 mm
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Other:
- board outline added: 103.5 x 70 mm

Commit message: adding stuff
Parts:
- removed A1: Adafruit_Feather_32u4_BluefruitLE, Module:Adafruit_Feather
- added U1: MCU_Seeed_XIAO_RP2040, ScottoKeebs_MCU:Seeed_XIAO_RP2040, F.Cu at (98.1, 70.1)
Routing:
- net x1: track 47.5 -> 156.5 mm, vias 0 -> 1
- net col0: track 161.3 -> 87.3 mm
- net row3: track 155.7 -> 83.9 mm
- net row2: track 118.3 -> 78.2 mm, vias 1 -> 0
- net y1: track 68.3 -> 101.5 mm
- net gnd: track 125.1 -> 156.8 mm
- net y2: track 56.9 -> 26.7 mm
- net row1: track 103.5 -> 76.3 mm, vias 1 -> 0
- net row0: track 43.3 -> 69.6 mm
- net 3.3v: track 192.3 -> 167.6 mm, vias 1 -> 0
- net Net-(D1-A): track 22.5 -> 12.5 mm
- net Net-(D11-A): track 23.6 -> 14.4 mm
- net Net-(D9-A): track 29.0 -> 25.5 mm
- net Net-(D12-A): track 9.57 -> 6.95 mm
- net col2: track 56.6 -> 54.1 mm
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
Commit message: finishing
Parts:
- U1: value MCU_Seeed_XIAO_RP2040 -> nRF52840_Featherwing; footprint ScottoKeebs_MCU:Seeed_XIAO_RP2040 -> Module:Adafruit_Feather
- moved U1 11.1 mm to (87.2, 67.9)
Connections:
- U1 pad 1: x1 -> unconnected-(U1-RST-Pad1)
- U1 pad 10: col0 -> unconnected-(U1-GPIOA5-Pad10)
- U1 pad 11: row3 -> unconnected-(U1-GPIOSCK-Pad11)
- U1 pad 12: 3.3v -> unconnected-(U1-GPIOMOSI-Pad12)
- U1 pad 13: gnd -> unconnected-(U1-GPIOMISO-Pad13)
- U1 pad 2: y1 -> 3.3v
- U1 pad 3: x2 -> unconnected-(U1-AREF-Pad3)
- U1 pad 4: y2 -> gnd
- U1 pad 5: row0 -> x1
- U1 pad 6: row1 -> y1
- U1 pad 7: row2 -> x2
- U1 pad 8: col2 -> y2
Routing:
- net x1: track 156.5 -> 46.7 mm, vias 1 -> 0
- net col0: track 87.3 -> 148.9 mm
- net 3.3v: track 167.6 -> 106.6 mm
- net gnd: track 156.8 -> 114.7 mm
- net col2: track 54.1 -> 95.2 mm
- net y1: track 101.5 -> 61.1 mm
- net row2: track 78.2 -> 42.7 mm, vias 0 -> 1
- net y2: track 26.7 -> 58.5 mm
- net row3: track 83.9 -> 61.5 mm
- net row0: track 69.6 -> 50.5 mm
- net row1: track 76.3 -> 63.2 mm
- net Net-(D12-A): track 6.95 -> 12.5 mm
- net x2: track 36.4 -> 39.6 mm
- net Net-(D9-A): track 25.5 -> 23.3 mm

Commit message: finding better switch
Routing:
- net Net-(D9-A): track 23.3 -> 55.2 mm
- net col2: track 95.2 -> 86.8 mm
- net col0: track 148.9 -> 154.1 mm
Changed lines of the file:
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@@
 	)
 	(segment
-		(start 132.098 83.5)
-		(end 140.5 83.5)
+		(start 128.899 80.301)
+		(end 126.799 80.301)
+		(width 0.2)
+		(layer "F.Cu")
+		(net 1)
+	)
+	(segment
+		(start 135.699 75.2359)
+		(end 135.699 71.699)
+		(width 0.2)
+		(layer "F.Cu")
+		(net 1)
+	)
+	(segment
+		(start 142.6349 75.2329)
+		(end 142.6349 79.8349)
+		(width 0.2)
+		(layer "F.Cu")
+		(net 1)
+	)
+	(segment
+		(start 126.799 80.301)
+		(end 126.799 78.699)
 		(width 0.2)
 		(layer "F.Cu")
@@
 	)
 	(segment
+		(start 126.799 78.699)
+		(end 132.2359 78.699)
+		(width 0.2)
+		(layer "F.Cu")
+		(net 1)
+	)
+	(segment
+		(start 132.2359 78.699)
+		(end 135.699 75.2359)
+		(width 0.2)
+		(layer "F.Cu")
+		(net 1)
+	)
+	(segment
+		(start 135.699 71.699)
+		(end 139.101 71.699)
+		(width 0.2)
+		(layer "F.Cu")
+		(net 1)
+	)
+	(segment
+		(start 142.6349 79.8349)
+		(end 146.3 83.5)
+		(width 0.2)
+		(layer "F.Cu")
+		(net 1)
+	)
+	(segment
+		(start 139.101 71.699)
+		(end 142.6349 75.2329)
+		(width 0.2)
+		(layer "F.Cu")
+		(net 1)
+	)
+	(segment
 		(start 118.62 87)
 		(end 128.598 87)
@@
 	)
 	(segment
+		(start 132.098 83.5)
+		(end 128.899 80.301)
+		(width 0.2)
+		(layer "F.Cu")
+		(net 1)
+	)
+	(segment
 		(start 87.48 78.06)
 		(end 87.48 78.177049)
@@
 	)
 	(segment
-		(start 66.2 116.2)
-		(end 63 113)
-		(width 0.2)
-		(layer "F.Cu")
-		(net 3)
-	)
-	(segment
-		(start 75 109.1)
-		(end 75 113)
+		(start 57.2 114.498)
+		(end 57.2 113)
 		(width 0.2)
 		(layer "F.Cu")
@@
 	)
 	(segment
-		(start 63 110.5)
-		(end 66.1 107.4)
+		(start 66.2 118.5)
+		(end 66.2 116.2)
 		(width 0.2)
 		(layer "F.Cu")
@@
 	)
 	(segment
-		(start 71.9 106)
-		(end 75 109.1)
+		(start 72 116)
+		(end 66.4 116)
+		(width 0.2)
+		(layer "F.Cu")
+		(net 3)
+	)
+	(segment
+		(start 66.2 118.5)
+		(end 61.202 118.5)
 		(width 0.2)
 		(layer "F.Cu")
@@
 	(segment
 		(start 66.2 120)
-		(end 66.2 116.2)
+		(end 66.2 118.5)
+		(width 0.2)
+		(layer "F.Cu")
+		(net 3)
+	)
+	(segment
+		(start 72.4 113)
+		(end 75 113)
 		(width 0.2)
 		(layer "F.Cu")
@@
 	)
 	(segment
-		(start 72 120)
-		(end 72 116)
-		(width 0.2)
-		(layer "F.Cu")
-		(net 3)
-	)
-	(segment
 		(start 53.064499 75.001549)
 		(end 57.2 79.13705)
@@
 	)
 	(segment
-		(start 63 113)
-		(end 63 110.5)
-		(width 0.2)
-		(layer "F.Cu")
-		(net 3)
-	)
-	(segment
-		(start 66.1 107.4)
-		(end 66.1 106)
+		(start 66.1 106.7)
+		(end 72.4 113)
+		(width 0.2)
+		(layer "F.Cu")
+		(net 3)
+	)
+	(segment
+		(start 66.4 116)
+		(end 66.2 116.2)
+		(width 0.2)
+		(layer "F.Cu")
+		(net 3)
+	)
+	(segment
+		(start 66.1 106)
+		(end 66.1 106.7)
+		(width 0.2)
+		(layer "F.Cu")
+		(net 3)
+	)
+	(segment
+		(start 61.202 118.5)
+		(end 57.2 114.498)
 		(width 0.2)
 		(layer "F.Cu")
@@
 	)
 	(segment
-		(start 140.002 86.5)
-		(end 131.6 86.5)
-		(width 0.2)
-		(layer "F.Cu")
-		(net 21)
-	)
-	(segment
