File: PCB/controller/controller.kicad_pcb (KiCad board)
At the start: 2 copper layers, 103.5 x 70 mm, 19 parts, among them U1 nRF52840_Featherwing, X1 Switch, Y1 Switch

Commit message: firmwere
Parts:
- removed U1: nRF52840_Featherwing, Module:Adafruit_Feather
- added U2: Adafruit-Feather-RP2040, Module:Adafruit_Feather, F.Cu at (87.2, 67.8)
