File: PCB/controller/controller.kicad_sch (KiCad schematic)
At the start: 14 parts, among them U1 Raspberry_Pi_Pico, X1 Switch, Y1 Switch

Commit message: doin stuffs
Parts:
- removed U1: Raspberry_Pi_Pico, ScottoKeebs_MCU:Raspberry_Pi_Pico, symbol ScottoKeebs:MCU_Raspberry_Pi_Pico
- added A1: Adafruit_Feather_32u4_BluefruitLE, Module:Adafruit_Feather, symbol MCU_Module:Adafruit_Feather_32u4_BluefruitLE
- added D1, D10, D11, D12, D2, D3, D4, D5, D6, D7, D8, D9: 1N4148, Diode_THT:D_DO-35_SOD27_P7.62mm_Horizontal, symbol Diode:1N4148
- added R1, R2: THB001P, ScottoKeebs_Miscellaneous:THB001P_CNK, symbol 2025-05-29_23-49-57:THB001P
Connections:
- net at B1.1: now also D_right1.1, ZL1.1, A1.23 (D11)
- net at B1.2: now also D10.2 (A)
- net at A2.1: now also D_UP1.1, L1.1, A1.22 (D10)
- net at A2.2: now also D9.2 (A)
- net at ZR1.1: now also D_Left1.1, Y1.1, A1.25 (D13)
- net at ZR1.2: now also D8.2 (A)
- net at R1.1: now also D_Down1.1, X1.1, A1.24 (D12)
- net at R1.2: now also D7.2 (A)
- net at Y1.2: now also D12.2 (A)
- net at D_Down1.2: now also D3.2 (A)
- net at ZL1.2: now also D6.2 (A)
- net at D_right1.2: now also D2.2 (A)
- net at D_Left1.2: now also D4.2 (A)
- net at D_UP1.2: now also D1.2 (A)
- net at X1.2: now also D11.2 (A)
- net at L1.2: now also D5.2 (A)
- new net: A1.19 (D5), D10.1 (K), D11.1 (K), D12.1 (K), D9.1 (K)
- new net: A1.2 (3V3), R1.1, R1.1', R2.1, R2.1'
- new net: A1.20 (D6), D5.1 (K), D6.1 (K), D7.1 (K), D8.1 (K)
- new net: A1.21 (D9), D1.1 (K), D2.1 (K), D3.1 (K), D4.1 (K)
- new net: A1.4 (GND), R1.2, R1.2', R2.2, R2.2'
- new net: A1.5 (A0), R2.3
- new net: A1.6 (A1), R2.3'
- new net: A1.7 (A2), R1.3
- new net: A1.8 (A3), R1.3'
Other:
- moved on the sheet: A2, B1, BT1, D_Down1, D_Left1, D_UP1, D_right1, L1, R1, X1, Y1, ZL1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

Commit message: more work
Parts:
- removed BT1: Battery_Cell, Battery:BatteryHolder_Bulgin_BX0034_1xAAA, symbol Device:Battery_Cell
- renumbered R1 to stick1, R2 to stick2
Connections:
- net col0: now reaches A1.23 (D11), D_right1.1
- net col0: now also D_Down1.1, D_Left1.1, D_UP1.1; no longer B1.1, ZL1.1
- net 3.3v: now reaches A1.2 (3V3), stick1.1, stick1.1', stick2.1, stick2.1'
- net col1: now reaches A1.24 (D12), R1.1
- net col1: now also L1.1, ZL1.1, ZR1.1; no longer D_Down1.1, X1.1
- net col2: now reaches A1.25 (D13), Y1.1
- net col2: now also A2.1, B1.1, X1.1; no longer D_Left1.1, ZR1.1
- net gnd: now reaches A1.4 (GND), stick1.2, stick1.2', stick2.2, stick2.2'
- net x1: now reaches A1.5 (A0), stick2.3
- net y1: now reaches A1.6 (A1), stick2.3'
- net x2: now reaches A1.7 (A2), stick1.3
- net y2: now reaches A1.8 (A3), stick1.3'
- new net row0: A1.19 (D5), D1.1 (K), D5.1 (K), D9.1 (K)
- new net row1: A1.20 (D6), D10.1 (K), D2.1 (K), D6.1 (K)
- new net row2: A1.21 (D9), D11.1 (K), D3.1 (K), D7.1 (K)
- new net row3: A1.22 (D10), D12.1 (K), D4.1 (K), D8.1 (K)
Other:
- moved on the sheet: A1, A2, B1, D1, D10, D11, D12, D2, D3, D4, D5, D6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

Commit message: finding that I need to change micro Controller
Parts:
- removed A1: Adafruit_Feather_32u4_BluefruitLE, Module:Adafruit_Feather, symbol MCU_Module:Adafruit_Feather_32u4_BluefruitLE
- added U1: RP2040_Pro_Micro, ScottoKeebs_MCU:RP2040_Pro_Micro, symbol ScottoKeebs:MCU_RP2040_Pro_Micro
Changed lines of the file:
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@@
-	)
-	(symbol
-		(lib_id "MCU_Module:Adafruit_Feather_32u4_BluefruitLE")
-		(at 207.01 55.88 0)
-		(unit 1)
-		(exclude_from_sim no)
-		(in_bom yes)
-		(on_board yes)
-		(dnp no)
-		(fields_autoplaced yes)
-		(property "Reference" "A1"
-			(at 209.1533 88.9 0)
-			(effects
-				(font
-					(size 1.27 1.27)
-				)
-				(justify left)
-			)
-		)
-		(property "Value" "Adafruit_Feather_32u4_BluefruitLE"
-			(at 209.1533 91.44 0)
-			(effects
-				(font
-					(size 1.27 1.27)
-				)
-				(justify left)
-			)
-		)
-		(property "Footprint" "Module:Adafruit_Feather"
-			(at 209.55 90.17 0)
-			(effects
-				(font
-					(size 1.27 1.27)
-					(italic yes)
-				)
-				(justify left)
-				(hide yes)
-			)
-		)
-		(property "Datasheet" "https://cdn-learn.adafruit.com/downloads/pdf/adafruit-feather-32u4-bluefruit-le.pdf"
-			(at 207.01 50.8 0)
-			(effects
-				(font
-					(size 1.27 1.27)
-				)
-				(hide yes)
-			)
-		)
-		(property "Description" "Microcontroller module with ATmega32u4 MCU and bluetooth"
-			(at 207.01 55.88 0)
-			(effects
-				(font
-					(size 1.27 1.27)
-				)
-				(hide yes)
-			)
-		)
-		(pin "5"
-		)
-		(pin "28"
-		)
-		(pin "8"
-		)
-		(pin "26"
-		)
-		(pin "19"
-		)
-		(pin "22"
-		)
-		(pin "24"
-		)
-		(pin "12"
-		)
-		(pin "15"
-		)
-		(pin "13"
-		)
-		(pin "20"
-		)
-		(pin "21"
-		)
-		(pin "1"
-		)
-		(pin "2"
-		)
-		(pin "11"
-		)
-		(pin "17"
-		)
-		(pin "18"
-		)
-		(pin "25"
-		)
-		(pin "14"
-		)
-		(pin "4"
-		)
-		(pin "23"
-		)
-		(pin "16"
-		)
-		(pin "27"
-		)
-		(pin "3"
-		)
-		(pin "6"
-		)
-		(pin "7"
-		)
-		(pin "10"
-		)
-		(pin "9"
-		)
-		(instances
-			(project ""
-				(path "/fd08eec5-01fb-42e9-ad15-054787276245"
-					(reference "A1")
-					(unit 1)
-				)
-			)
-		)
 	)
 	(symbol
@@
 					(unit 1)
 				)
+			)
+		)
+	)
+	(symbol
+		(lib_id "ScottoKeebs:MCU_RP2040_Pro_Micro")
+		(at 208.28 121.92 0)
+		(unit 1)
+		(exclude_from_sim no)
+		(in_bom yes)
+		(on_board yes)
+		(dnp no)
+		(fields_autoplaced yes)
+		(property "Reference" "U1"
+			(at 208.28 100.33 0)
+			(effects
+				(font
+					(size 1.524 1.524)
+				)
+			)
+		)
+		(property "Value" "RP2040_Pro_Micro"
+			(at 208.28 102.87 0)
+			(effects
+				(font
+					(size 1.524 1.524)
+				)
+			)
+		)
+		(property "Footprint" "ScottoKeebs_MCU:RP2040_Pro_Micro"
+			(at 208.28 153.416 0)
+			(effects
+				(font
+					(size 1.524 1.524)
+				)
+				(hide yes)
+			)
+		)
+		(property "Datasheet" ""
+			(at 234.95 185.42 90)
+			(effects
+				(font
+					(size 1.524 1.524)
+				)
+				(hide yes)
+			)
+		)
+		(property "Description" ""
+			(at 208.28 121.92 0)
+			(effects
+				(font
+					(size 1.27 1.27)
+				)
+				(hide yes)
+			)
+		)
+		(pin "6"
+		)
+		(pin "8"
+		)
+		(pin "15"
+		)
+		(pin "11"
+		)
+		(pin "1"
+		)
+		(pin "4"
+		)
+		(pin "17"
+		)
+		(pin "14"
+		)
+		(pin "9"
+		)
+		(pin "2"
+		)
+		(pin "12"
+		)
+		(pin "16"
+		)
+		(pin "28"
+		)
+		(pin "13"
+		)
+		(pin "3"
+		)
+		(pin "30"
+		)
+		(pin "27"
+		)
+		(pin "10"
+		)
+		(pin "5"
+		)
+		(pin "7"
+		)
+		(pin "18"
+		)
+		(pin "31"
+		)
+		(pin "29"
+		)
+		(pin "26"
+		)
+		(pin "25"
+		)
+		(pin "24"
+		)
+		(pin "19"
+		)
+		(pin "21"
+		)
+		(pin "22"
+		)
+		(pin "20"
+		)
+		(pin "23"
+		)
+		(instances
+			(project ""
+				(path "/fd08eec5-01fb-42e9-ad15-054787276245"
+					(reference "U1")
+					(unit 1)
+				)

Commit message: adding stuff
Parts:
- removed D5, D6, D7, D8: 1N4148, Diode_THT:D_DO-35_SOD27_P7.62mm_Horizontal, symbol Diode:1N4148
- removed L1, R1, ZL1, ZR1: Switch, Button_Switch_SMD:SW_Push_1P1T_NO_CK_KSC6xxJ, symbol ScottoKeebs:Placeholder_Switch
- removed U1: RP2040_Pro_Micro, ScottoKeebs_MCU:RP2040_Pro_Micro, symbol ScottoKeebs:MCU_RP2040_Pro_Micro
- added U1: MCU_Seeed_XIAO_RP2040, ScottoKeebs_MCU:Seeed_XIAO_RP2040, symbol ScottoKeebs:MCU_Seeed_XIAO_RP2040
Connections:
- net 3.3v: now also U1.12 (3V3)
- net col0: now also U1.10 (PA5_A9_D9_MISO)
- net col2: now also U1.8 (PB09_A7_D7_RX)
- net gnd: now also U1.13 (GND)
- net row0: now also U1.5 (PA8_A4_D4_SDA)
- net row1: now also U1.6 (PA9_A5_D5_SCL)
- net row2: now also U1.7 (PB08_A6_D6_TX)
- net row3: now also U1.11 (PA6_A10_D10_MOSI)
- net x1: now also U1.1 (PA02_A0_D0)
- net x2: now also U1.3 (PA10_A2_D2)
- net y1: now also U1.2 (PA4_A1_D1)
- net y2: now also U1.4 (PA11_A3_D3)

Commit message: finishing
Parts:
- removed U1: MCU_Seeed_XIAO_RP2040, ScottoKeebs_MCU:Seeed_XIAO_RP2040, symbol ScottoKeebs:MCU_Seeed_XIAO_RP2040
- added U1: nRF52840_Featherwing, Module:Adafruit_Feather, symbol dumb:nRF52840_Featherwing
Connections:
- net 3.3v: now also U1.2 (3V)
- net col0: now also U1.21 (GPIO9)
- net col2: now also U1.20 (GPIO6)
- net gnd: now also U1.4 (GND)
- net row0: now also U1.25 (GPIO13)
- net row1: now also U1.24 (GPIO12)
- net row2: now also U1.23 (GPIO11)
- net row3: now also U1.22 (GPIO10)
- net x1: now also U1.5 (GPIOA0)
- net x2: now also U1.7 (GPIOA2)
- net y1: now also U1.6 (GPIOA1)
- net y2: now also U1.8 (GPIOA3)

Commit message: firmwere
Parts:
- removed U1: nRF52840_Featherwing, Module:Adafruit_Feather, symbol dumb:nRF52840_Featherwing
- added U2: Adafruit-Feather-RP2040, Module:Adafruit_Feather, symbol Adafruit-Feather-RP2040:Adafruit-Feather-RP2040
Connections:
- net 3.3v: now also U2.2 (3.3V)
- net col0: now also U2.21 (D9/GPIO9)
- net col2: now also U2.20 (D6/GPIO8)
- net gnd: now also U2.4 (GND)
- net row0: now also U2.25 (D13/GPIO13)
- net row1: now also U2.24 (D12/GPIO12)
- net row2: now also U2.23 (D11/GPIO11)
- net row3: now also U2.22 (D10/GPIO10)
- net x1: now also U2.5 (A0/GPIO26)
- net x2: now also U2.7 (A2/GPIO28)
- net y1: now also U2.6 (A1/GPIO27)
- net y2: now also U2.8 (A3/GPIO29)
